File: EDA/EDA/EDA.sch (KiCad schematic (older format))
At the start: 28 parts

Commit message: more work on PCB routing
Parts:
- removed TP?: MISC_GPIO1, symbol Connector:TestPoint
- removed TP?: MISC_GPIO2, symbol Connector:TestPoint
- removed TP?: MISC_GPIO0, symbol Connector:TestPoint
- removed TP?: 1V8_OUT, symbol Connector:TestPoint
- C2, C3, C4, C5: renamed from C?; footprint (none) -> Capacitor_SMD:C_0603_1608Metric
- J1, J3: renamed from J?; footprint (none) -> Connector_PinHeader_1.27mm:PinHeader_2x03_P1.27mm_Vertical
- J2: renamed from J?; footprint (none) -> Connector_PinHeader_1.27mm:PinHeader_1x04_P1.27mm_Vertical
- JP1: renamed from JP?; footprint (none) -> Jumper:SolderJumper-2_P1.3mm_Open_Pad1.0x1.5mm
- R1, R2, R4: renamed from R?; footprint (none) -> Resistor_SMD:R_0603_1608Metric
- R3: renamed from R?; value 1 kΩ -> 100 Ω; footprint (none) -> Resistor_SMD:R_0603_1608Metric
- TP1, TP2, TP4, TP5, TP6: renamed from TP?; footprint (none) -> TestPoint:TestPoint_Pad_1.0x1.0mm
- U2: renamed from U?; footprint (none) -> EDA:DHVQFN14
- U3: renamed from U?; footprint (none) -> Package_TO_SOT_SMD:SOT-363_SC-70-6
- U5: renamed from U?; footprint (none) -> EDA:XM132
- gave numbers to parts that had none: 4
Connections:
- net GND: now also Y1.2, Y1.4
- net MISO: now also U2.3 (1Y); no longer U2.6 (2Y)
- net MOSI: now also U2.5 (2A); no longer U2.2 (1A)
- net RDR_RX: now also U2.2 (1A); no longer U2.5 (2A)
- net RDR_TX: now also U2.6 (2Y); no longer U2.3 (1Y)
- net VACC: now also U1.24 (PC1); no longer U1.11 (PD7)
- net at U1.7 (XTAL1/PB6), Y1.1: now also C4.1
- net at U1.8 (XTAL2/PB7), Y1.3: now also C3.1
- no-connect marks 3 -> 7
Other:
- moved on the sheet: C1, C3, C4, C5, J3, U3, U4
